File: NeoGB-Printer-ESP32/NeoGB-Printer-ESP32.kicad_sch (KiCad schematic)
At the start: 76 parts, among them J1 USB_C_Receptacle_USB2.0, J2 Conn_01x02_Shielded, J3 Micro_SD_Card_Det1, J4 Conn_01x30, J5 GameBoy_LinkPort, Q1 DMG3415U, Q2 BSS138, Q3 BSS138, Q4 BSS138, Q7 UMH3N, SW1 SW_Push_DPDT, SW2 SW_MEC_5E, SW3 SW_MEC_5E, SW4 SW_MEC_5E, U1 ESP32-WROOM-32D, U2 CP2102N-Axx-xQFN28, U3 USBLC6-2P6, U4 TPS63802DLAR, U5 MCP73831-2-OT

Commit message: more schematic and layout
Parts:
- removed D2: D_Schottky, Diode_SMD:D_SOD-123F, symbol Device:D_Schottky
- removed J4: Conn_01x30, Bongo-Cat-Fidget-Toy:sh1106-1.3inch-oled, symbol Connector_Generic:Conn_01x30
- removed JP1: SolderJumper_2_Bridged, Jumper:SolderJumper-2_P1.3mm_Bridged_RoundedPad1.0x1.5mm, symbol Jumper:SolderJumper_2_Bridged
- removed Q7: UMH3N, Package_TO_SOT_SMD:SOT-363_SC-70-6, symbol Transistor_BJT:UMH3N
- removed R15: 100k, Resistor_SMD:R_0603_1608Metric, symbol Device:R_Small_US
- removed R16, R17: 4.7k, Resistor_SMD:R_0603_1608Metric, symbol Device:R_Small_US
- removed R18: JMP, Resistor_SMD:R_0603_1608Metric, symbol Device:R_Small_US
- removed R19: 390k, Resistor_SMD:R_0603_1608Metric, symbol Device:R_Small_US
- removed R33, R34: 10k, Resistor_SMD:R_0603_1608Metric, symbol Device:R_Small_US
- removed SW1: SW_Push_DPDT, mod:SS-3235S-L2, symbol Switch:SW_Push_DPDT
- removed SW3, SW4: SW_MEC_5E, Bongo-Cat-Fidget-Toy:SW_SKRPACE010, symbol Switch:SW_MEC_5E
- removed U1: ESP32-WROOM-32D, RF_Module:ESP32-WROOM-32D, symbol RF_Module:ESP32-WROOM-32D
- removed U2: CP2102N-Axx-xQFN28, Package_DFN_QFN:QFN-28-1EP_5x5mm_P0.5mm_EP3.35x3.35mm, symbol Interface_USB:CP2102N-Axx-xQFN28
- added C17: 10u, Capacitor_SMD:C_0603_1608Metric, symbol Device:C_Small
- added C18: 22u, Capacitor_SMD:C_0603_1608Metric, symbol Device:C_Small
- added C19: 1u, Capacitor_SMD:C_0402_1005Metric, symbol Device:C_Small
- added C25: 100n, Capacitor_SMD:C_0603_1608Metric, symbol Device:C_Small
- added C29: 100n, Capacitor_SMD:C_0402_1005Metric, symbol Device:C_Small
- added D2: WS2812B-2020, LED_SMD:LED_WS2812B-2020_PLCC4_2.0x2.0mm, symbol LED:WS2812B-2020
- added J6: Conn_01x03_MountingPin, Connector_JST:JST_SH_SM03B-SRSS-TB_1x03-1MP_P1.00mm_Horizontal, symbol Connector_Generic_MountingPin:Conn_01x03_MountingPin
- added J7: Conn_01x04, mod:OLED_SSD1306_128x32_0.91, symbol Connector_Generic:Conn_01x04
- added L2: 0.47uH, Inductor_SMD_Wurth:L_Wurth_WE-LQSH-2010, symbol Device:L
- added R32, R35, R36, R39: 0, Resistor_SMD:R_0402_1005Metric, symbol Device:R_Small_US
- added R37: 806k, Resistor_SMD:R_0402_1005Metric, symbol Device:R_Small_US
- added R38: 91k, Resistor_SMD:R_0402_1005Metric, symbol Device:R_Small_US
- added R40: 27.4, Resistor_SMD:R_0402_1005Metric, symbol Device:R_Small_US
- added R41, R42: 100, Resistor_SMD:R_0402_1005Metric, symbol Device:R_Small_US
- added R43, R44: 1k, Resistor_SMD:R_0402_1005Metric, symbol Device:R_Small_US
- added R45: DNI, Resistor_SMD:R_0402_1005Metric, symbol Device:R_Small_US
- added R46, R47: 4.7k, Resistor_SMD:R_0603_1608Metric, symbol Device:R_Small_US
- added SW3: SW_SPDT_321, Bongo-Cat-Fidget-Toy:SW-SMD_SK-3245S-L1-A-1, symbol Switch:SW_SPDT_321
- added SW5, SW6: SW_MEC_5E, mod:SW_SKRPACE010, symbol Switch:SW_MEC_5E
- added U1: RP2040, Package_DFN_QFN:QFN-56-1EP_7x7mm_P0.4mm_EP3.2x3.2mm, symbol MCU_RaspberryPi:RP2040
- added U2: W25Q32JVSS, Package_SON:Winbond_USON-8-1EP_3x2mm_P0.5mm_EP0.2x1.6mm, symbol Memory_Flash:W25Q32JVSS
- added U6: TPS63802DLAR, mod:VREG_TPS63802DLAR, symbol mod:TPS63802DLAR
- added Y1: 12MHZ, Crystal:Crystal_SMD_3225-4Pin_3.2x2.5mm, symbol Device:Crystal_GND24_Small
- C11: value 100n -> 1u; footprint Capacitor_SMD:C_0603_1608Metric -> Capacitor_SMD:C_0402_1005Metric; LCSC C478888 -> (none)
- C12, C16: footprint Capacitor_SMD:C_0603_1608Metric -> Capacitor_SMD:C_0402_1005Metric; LCSC C478888 -> (none)
- C13: value 10u -> 100n; footprint Capacitor_SMD:C_0603_1608Metric -> Capacitor_SMD:C_0402_1005Metric; LCSC C95839 -> (none)
- C14: value 100n -> 27p; LCSC C478888 -> C107045
- C15: value 10u -> 27p; LCSC C95839 -> C107045
- C3, C5, C7, C8: value 2.2u -> 100n; footprint Capacitor_SMD:C_0603_1608Metric -> Capacitor_SMD:C_0402_1005Metric; LCSC C23630 -> (none)
- C4: value 4.7u -> 100n; footprint Capacitor_SMD:C_0603_1608Metric -> Capacitor_SMD:C_0402_1005Metric; LCSC C23630 -> (none)
- C6: value 2.2u -> 1u; footprint Capacitor_SMD:C_0603_1608Metric -> Capacitor_SMD:C_0402_1005Metric; LCSC C23630 -> (none)
- J3: footprint mod:J_sd_micro_socket -> mod:J_sd_micro_socket_no_holes
- L1: footprint Inductor_SMD:L_Chilisin_BMRB00050512 -> Inductor_SMD_Wurth:L_Wurth_WE-LQSH-2010; LCSC C329374 -> C89446
- R1, R2: footprint Resistor_SMD:R_0603_1608Metric -> Resistor_SMD:R_0402_1005Metric; LCSC C407575 -> (none)
- R31: value 100k -> 27.4; footprint Resistor_SMD:R_0603_1608Metric -> Resistor_SMD:R_0402_1005Metric; LCSC C25803 -> C274349
- R4: footprint Resistor_SMD:R_0603_1608Metric -> Resistor_SMD:R_0402_1005Metric; symbol Device:R -> Device:R_Small_US; LCSC C95177 -> (none)
- R5, R6: footprint Resistor_SMD:R_0603_1608Metric -> Resistor_SMD:R_0402_1005Metric
- R7: footprint Resistor_SMD:R_0603_1608Metric -> Resistor_SMD:R_0402_1005Metric; LCSC C2684557 -> (none)
- R9: footprint Resistor_SMD:R_0603_1608Metric -> Resistor_SMD:R_0402_1005Metric; LCSC C95177 -> (none)
Connections:
- net GPIO0 is gone; now on net GND: C12.2
- net LIPO_IN is gone; now on net +BATT: C9.2, J2.1 (Pin_1), U5.3 (V_{BAT})
- net RESET is gone; now on net GND: C11.2
- net VBUS_IN is gone; now on net VBUS: C10.2, D5.2 (A), J1.A4 (VBUS), J1.A9 (VBUS), J1.B4 (VBUS), J1.B9 (VBUS), U3.5 (VBUS), U5.4 (V_{DD})
- net +3V3: now also C12.1, C13.1, C16.1, C3.1, C4.1, C5.1, C6.1, C19.1, C29.1, J7.3 (Pin_3), R45.1, R46.1, R47.1, U1.1 (IOVDD), U1.10 (IOVDD), U1.22 (IOVDD), U1.33 (IOVDD), U1.42 (IOVDD), U1.43 (ADC_AVDD), U1.44 (VREG_IN), U1.48 (USB_VDD), U1.49 (IOVDD), U2.8 (VCC)
- net 3V3: now also D2.4 (VDD); no longer C3.2, C6.2
- net GB_MISO: now also U1.5 (GPIO3)
- net GB_MOSI: now also U1.6 (GPIO4)
- net GB_SCK: now also U1.4 (GPIO2)
- net GND: now also C13.2, C16.2, C3.2, C4.2, C5.2, C6.2, C7.2, C8.2, C17.2, C18.2, C19.2, C25.2, C29.2, D2.2 (VSS), J6.2 (Pin_2), J6.MP (MountPin), J7.4 (Pin_4), R36.1, R38.2, SW5.1, SW5.2, SW6.1, SW6.2, U1.19 (TESTEN), U1.57 (GND), U2.4 (GND), U6.3 (AGND), U6.8 (GND), Y1.2, Y1.4; no longer C11.1, C12.1, C13.1, C16.1, C3.1, C4.1, C6.1, C7.1
- net PUSH_BTN: now also U1.15 (GPIO12)
- net SD_DET: now also U1.9 (GPIO7)
- net SPI_1_CS: now also U1.12 (GPIO9)
- net SPI_1_MISO: now also U1.11 (GPIO8)
- net SPI_1_MOSI: now also U1.14 (GPIO11)
- net SPI_1_SCK: now also U1.13 (GPIO10)
- net USB_D_N: now also R40.1
- net USB_D_P: now also R31.1
- net VBUS: no longer C13.2, C14.2, C15.2, C16.2, R20.1, R21.1, R24.1, R31.2
- net at D1.1 (K), Q1.2 (S): now also SW3.2 (B); no longer R4.1
- net at U4.7 (L2): now also L1.2; no longer L1.1
- net at U4.9 (L1): now also L1.1; no longer L1.2
- net +1V1: now reaches C8.1
- net +1V1: now also C11.1, C7.1, U1.23 (DVDD), U1.45 (VREG_VOUT), U1.50 (DVDD)
- new net: R35.1, R36.2, U6.2 (MODE)
- new net: C17.1, R32.2, R35.2, U6.1 (EN), U6.10 (VIN)
- new net: L2.1, U6.9 (L1)
- new net: L2.2, U6.7 (L2)
- new net: C18.1, R37.1, R39.1, U6.6 (VOUT)
- new net: R37.2, R38.1, U6.4 (FB)
- new net: C14.2, U1.20 (XIN), Y1.3
- new net: R32.1, R4.1, SW3.1 (C)
- new net: R40.2, U1.46 (USB_DM)
- new net: R41.2, U1.24 (SWCLK)
- new net: C15.2, R43.1, Y1.1
- new net: R43.2, U1.21 (XOUT)
- new net: R42.2, U1.25 (SWD)
- new net: R31.2, U1.47 (USB_DP)
- new net +5V: R20.1, R21.1, R24.1, R39.2
- new net LED0: D2.3 (DIN), U1.27 (GPIO16)
- new net MCU_SWCLK: J6.1 (Pin_1), R41.1
- new net MCU_SWD: J6.3 (Pin_3), R42.1
- new net OLED_SCL: J7.2 (Pin_2), R47.2, U1.3 (GPIO1)
- new net OLED_SDA: J7.1 (Pin_1), R46.2, U1.2 (GPIO0)
- new net QSPI_SCLK: U1.52 (QSPI_SCLK), U2.6 (CLK)
- new net QSPI_SD0: U1.53 (QSPI_SD0), U2.5 (DI(IO0))
- new net QSPI_SD1: U1.55 (QSPI_SD1), U2.2 (DO(IO1))
- new net QSPI_SD2: U1.54 (QSPI_SD2), U2.3 (IO2)
- new net QSPI_SD3: U1.51 (QSPI_SD3), U2.7 (IO3)
- new net QSPI_SS: R44.2, R45.2, U1.56 (QSPI_SS), U2.1 (~{CS})
- new net RUN: C25.1, SW6.3 (K), SW6.4 (A), U1.26 (RUN)
- new net ~{USB_BOOT}: R44.1, SW5.3 (K)
- no-connect marks 21 -> 8
Other:
- note removed: "1 NC(GND) 2 C2P 3 C2N 4 C1P 5 C1N 6 VBAT 7 VSS 8 VSS 9 VDD 10 BS0 11 BS1 12 BS2 13 CS 14 RES 15 DC 16 RW 17 ERD 18 D0 19 D1 20 D2 21 D3 22 D4 23 D5 24 D6 25 D7 26 IREF 27 VCOMH 28 VCC 29 NC 30 NC(GND)"
- moved on the sheet: C1, C2, D1, D3, J5, Q1, Q2, Q3, Q4, R10, R20, R21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
