File: hardware/yet-another-pico-gb-printer/yet-another-pico-gb-printer.kicad_sch (KiCad schematic)
At the start: 90 parts, among them J1 USB_C_Receptacle_USB2.0, J2 Conn_01x02_Shielded, J3 Micro_SD_Card_Det1, J5 GameBoy_LinkPort, J6 Conn_01x03_MountingPin, J7 Conn_01x04, Q1 DMG3415U, Q2 BSS138, Q3 BSS138, Q4 BSS138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

Commit message: schematics and layout improvements
Parts:
- added C20: 100n, Capacitor_SMD:C_0402_1005Metric, symbol Device:C_Small
- SW2: footprint Bongo-Cat-Fidget-Toy:SW_SKRPACE010 -> yet-another-pico-gb-printer:SW-SMD_4P-L5.2-W5.2-P3.70-LS6.4; LCSC C139797 -> C2686853
Connections:
- net +3V3: now also C20.1
- net GND: now also C20.2
- net ~{USB_BOOT}: now also SW5.4 (A)
Other:
- moved on the sheet: C11, C12, C13, C16, C19, C3, C4, C5, C6, C7, C8

Commit message: schematics and layout improvements
Parts:
- added H1, H2, H3, H4: M2, MountingHole:MountingHole_2.2mm_M2_Pad, symbol Mechanical:MountingHole_Pad_MP
Connections:
- net GND: now also H1.MP, H2.MP, H3.MP, H4.MP

Commit message: sent to fab
Parts:
- removed H1, H2, H3, H4: M2, MountingHole:MountingHole_2.2mm_M2_Pad, symbol Mechanical:MountingHole_Pad_MP
- removed R25: 10k, Resistor_SMD:R_0603_1608Metric, symbol Device:R_Small_US
- added R15, R16, R17, R18: 0, Resistor_SMD:R_0402_1005Metric, symbol Device:R_Small_US
- added R19: 10k, Resistor_SMD:R_0402_1005Metric, symbol Device:R_Small_US
- C11, C19, C6: LCSC (none) -> C14445
- C12, C13, C16, C20, C29, C3, C4, C5, C7, C8: LCSC (none) -> C60474
- C14, C15: LCSC C107045 -> C107002
- C25: LCSC C478888 -> C60474
- J5: footprint Gekkio_Connector:GameBoy_LinkPort_MGB_Horizontal -> yet-another-pico-gb-printer:GBA-LINK; now not fitted; now left out of the parts list
- J7, R46, R47: now left out of the parts list
- Q2, Q3, Q4: LCSC (none) -> C5337205
- R1, R2: LCSC (none) -> C105872
- R20, R21, R22, R23, R24, R29, R30: footprint Resistor_SMD:R_0603_1608Metric -> Resistor_SMD:R_0402_1005Metric; LCSC (none) -> C60490
- R26: footprint Resistor_SMD:R_0603_1608Metric -> Resistor_SMD:R_0402_1005Metric; LCSC (none) -> C145071
- R3: footprint Resistor_SMD:R_0603_1608Metric -> Resistor_SMD:R_0402_1005Metric; LCSC C103199 -> C60490
- R31, R40: LCSC C274349 -> C172043
- R32, R39, R4, R9: LCSC (none) -> C106231
- R35, R36, R5, R6: LCSC C95177 -> C106231
- R37: LCSC (none) -> C3016043
- R7: LCSC (none) -> C5126239
- SW3: footprint Bongo-Cat-Fidget-Toy:SW-SMD_SK-3245S-L1-A-1 -> yet-another-pico-gb-printer:SW-SMD_K3-1280S-L1; LCSC C405951 -> C223845
- U5: LCSC (none) -> C625600
Connections:
- net 3V3 is gone; now on net +3V3: D2.4 (VDD), SW2.3 (K), SW2.4 (A)
- net GB_SI: now also R16.1, R17.1; no longer J5.3 (SI)
- net GB_SO: now also R15.1, R18.1; no longer J5.2 (SO)
- net GND: now also R19.2
- net PUSH_BTN: now also R19.1
- net at R32.1, R4.1: now also SW3.3 (A); no longer SW3.1 (C)
- net PICO_USB_D_N: now reaches R40.2, U1.46 (USB_DM)
- net PICO_USB_D_P: now reaches R31.2, U1.47 (USB_DP)
- new net: J5.2 (SO), R15.2, R16.2
- new net: J5.3 (SI), R17.2, R18.2
Other:
- moved on the sheet: R31, R40
